File: neocera engr project/NEOCERA_jnr_project/NEOCERA_jnr_project.kicad_sch (KiCad schematic)
At the start: 0 parts

Commit message: microcontoller
microcontroller
Other:
- added sheet stepperstage-microcontroller (microcontroller.kicad_sch)
Changed lines of the file:
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@@
+	)
+	(sheet
+		(at 149.86 74.93)
+		(size 46.99 36.83)
+		(fields_autoplaced yes)
+		(stroke
+			(width 0.1524)
+			(type solid)
+		)
+		(fill
+			(color 0 0 0 0.0000)
+		)
+		(property "Sheetname" "stepperstage-microcontroller"
+			(at 149.86 74.2184 0)
+			(effects
+				(font
+					(size 1.27 1.27)
+				)
+				(justify left bottom)
+			)
+		)
+		(property "Sheetfile" "microcontroller.kicad_sch"
+			(at 149.86 112.3446 0)
+			(effects
+				(font
+					(size 1.27 1.27)
+				)
+				(justify left top)
+			)
+		)
+		(instances
+			(project "NEOCERA_jnr_project"
+				(path "/a8746ab6-0163-416c-99f9-0036ded73fc6"
+					(page "7")
+				)
+			)
+		)
 	)
 	(sheet
