File: NEOCERA_jnr_project/1224voltsdrivingoutputMOSFET.kicad_sch (KiCad schematic)
At the start: 20 parts, among them Q1 BSS138, Q10 BSS138, Q11 Q_PMOS_GSD, Q2 Q_PMOS_GSD, Q3 BSS138, Q4 Q_PMOS_GSD, Q5 BSS138, Q6 Q_PMOS_GSD

Commit message: bunch of edits
bunch of edits were done including DB37
Connections:
- net HV renamed +24V
- net hvcontrol1_controller renamed hvcontrol1_in
- net hvcontrol2_controller renamed hvcontrol2_in
- net hvcontrol3_controller renamed hvcontrol3_in
- net hvcontrol4_controller renamed hvcontrol4_in
Other:
- note added: "IS this to be 24V?"
- moved on the sheet: Q10, Q11, R39, R40, R41

Commit message: bunch
bunch
Connections:
- net hvcontrol1_in renamed hvcontrol1_microcontroller
- net hvcontrol2_in renamed hvcontrol2_microcontroller
- net hvcontrol3_in renamed hvcontrol3_microcontroller
- net hvcontrol4_in renamed hvcontrol4_microcontroller
- net hvout1_signal renamed hvout1_mboard
- net hvout2_signal renamed hvout2_mboard
- net hvout3_signal renamed hvout3_mboard
- net hvout4_signal renamed hvout4_mboard
Other:
- note removed: "IS this to be 24V?"
Changed lines of the file:
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@@
 		)
 	)
-	(text "IS this to be 24V?"
-		(exclude_from_sim no)
-		(at 76.708 59.436 0)
-		(effects
-			(font
-				(size 1.27 1.27)
-			)
-		)
-	)
-	(text "IS this to be 24V?"
-		(exclude_from_sim no)
-		(at 229.108 59.436 0)
-		(effects
-			(font
-				(size 1.27 1.27)
-			)
-		)
-	)
-	(text "IS this to be 24V?"
-		(exclude_from_sim no)
-		(at 171.958 59.436 0)
-		(effects
-			(font
-				(size 1.27 1.27)
-			)
-		)
-	)
-	(text "IS this to be 24V?"
-		(exclude_from_sim no)
-		(at 126.238 59.436 0)
-		(effects
-			(font
-				(size 1.27 1.27)
-			)
-		)
-	)
-	(global_label "hvout2_signal"
+	(global_label "hvout2_mboard"
 		(shape output)
 		(at 130.81 96.52 0)
@@
 		)
 	)
-	(global_label "hvcontrol3_in"
+	(global_label "hvcontrol3_microcontroller"
 		(shape input)
 		(at 148.59 110.49 180)
@@
 		)
 	)
-	(global_label "hvcontrol4_in"
+	(global_label "hvcontrol4_microcontroller"
 		(shape input)
 		(at 205.74 110.49 180)
@@
 		)
 	)
-	(global_label "hvout4_signal"
+	(global_label "hvout4_mboard"
 		(shape output)
 		(at 233.68 96.52 0)
@@
 		)
 	)
-	(global_label "hvout3_signal"
+	(global_label "hvout3_mboard"
 		(shape output)
 		(at 176.53 96.52 0)
@@
 		)
 	)
-	(global_label "hvout1_signal"
+	(global_label "hvout1_mboard"
 		(shape output)
 		(at 81.28 96.52 0)
@@
 		)
 		(property "Intersheetrefs" "${INTERSHEET_REFS}"
-			(at 90.615 96.52 0)
+			(at 94.6063 96.52 0)
 			(effects
 				(font
@@
 		)
 	)
-	(global_label "hvcontrol2_in"
+	(global_label "hvcontrol2_microcontroller"
 		(shape input)
 		(at 102.87 110.49 180)
@@
 		)
 	)
-	(global_label "hvcontrol1_in"
+	(global_label "hvcontrol1_microcontroller"
 		(shape input)
 		(at 53.34 110.49 180)
@@
 		)
 		(property "Intersheetrefs" "${INTERSHEET_REFS}"
-			(at 37.5946 110.49 0)
+			(at 24.7738 110.49 0)
 			(effects
 				(font
