File: NEOCERA_jnr_project/micro.kicad_sch (KiCad schematic)
At the start: 19 parts, among them J2 Conn_01x06_MountingPin, U13 BD48LxxG, U30 PIC18F45K50_QFP, Y1 ASV-xxxMHz

Commit message: changes
Parts:
- U13: value BD48LxxG -> MCP111T; footprint Package_TO_SOT_SMD:SOT-23 -> Package_TO_SOT_SMD:TSOT-23
Changed lines of the file:
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@@
 			)
 		)
-		(property "Value" "BD48LxxG"
+		(property "Value" "MCP111T"
 			(at 241.3 83.8199 0)
 			(effects
@@
 			)
 		)
-		(property "Footprint" "Package_TO_SOT_SMD:SOT-23"
+		(property "Footprint" "Package_TO_SOT_SMD:TSOT-23"
 			(at 236.22 69.85 0)
 			(effects
