File: NEOCERA_jnr_project/NEOCERA_jnr_project.kicad_pcb (KiCad board)
At the start: 2 copper layers, 42 parts, among them Q1 BSS138, Q13 BSS138, Q2 Q_PMOS_GSD, Q3 BSS138, Q4 Q_PMOS_GSD, Q5 BSS138, Q6 Q_PMOS_GSD, Q7 BSS138, Q8 BSS138, Q9 BSS138, U1 ICL3232, U2 ICL3232, U3 74AHCT1G126, U4 HCPL-2630, U5 HCPL-2630, U6 HCPL-2630, U7 HCPL-2630

Commit message: changes
Parts:
- removed C1, C10, C2, C3, C4, C5, C6, C7, C8, C9: 0.1uF, Capacitor_SMD:C_0603_1608Metric_Pad1.08x0.95mm_HandSolder
- removed Q1, Q13, Q3, Q5, Q7, Q8, Q9: BSS138, Package_TO_SOT_SMD:SOT-23_Handsoldering
- removed Q2, Q4, Q6: Q_PMOS_GSD, Package_TO_SOT_SMD:SOT-23_Handsoldering
- removed R1, R19, R2, R5, R6, R8, R9: 10k, Resistor_SMD:R_0603_1608Metric_Pad0.98x0.95mm_HandSolder
- removed R10: 100, Resistor_SMD:R_0603_1608Metric_Pad0.98x0.95mm_HandSolder
- removed R11, R12, R13, R17, R3, R4, R7: 1.5k, Resistor_SMD:R_0603_1608Metric_Pad0.98x0.95mm_HandSolder
- removed U1, U2: ICL3232, Package_SO:SOIC-16W_7.5x12.8mm_P1.27mm
- removed U3: 74AHCT1G126, Package_TO_SOT_SMD:SOT-23-5_HandSoldering
- removed U4, U5, U6, U7: HCPL-2630, Package_DIP:DIP-8_W7.62mm

Commit message: Ratnest
started working on rat nest.
Parts:
- added C1: 0.1uF, Capacitor_SMD:C_0603_1608Metric_Pad1.08x0.95mm_HandSolder, F.Cu at (131.6, 126.3)
- added C10: 0.1uF, Capacitor_SMD:C_0603_1608Metric_Pad1.08x0.95mm_HandSolder, F.Cu at (135.9, 136.3)
- added C11: 10uf 50V, Capacitor_SMD:C_0603_1608Metric_Pad1.08x0.95mm_HandSolder, F.Cu at (93.3, 74.5)
- added C12: 0.1uf, Capacitor_SMD:C_0603_1608Metric_Pad1.08x0.95mm_HandSolder, F.Cu at (93.3, 77.0)
- added C13: 0.1u, Capacitor_SMD:C_0603_1608Metric_Pad1.08x0.95mm_HandSolder, F.Cu at (93.3, 79.5)
- added C14: 0.1u, Capacitor_SMD:C_0603_1608Metric_Pad1.08x0.95mm_HandSolder, F.Cu at (93.3, 82.0)
- added C15: 10uf_50V, Capacitor_SMD:C_0603_1608Metric_Pad1.08x0.95mm_HandSolder, F.Cu at (93.3, 84.5)
- added C16: 0.1uf, Capacitor_SMD:C_0603_1608Metric_Pad1.08x0.95mm_HandSolder, F.Cu at (93.3, 87.0)
- added C17: 470uf, Capacitor_SMD:C_0603_1608Metric_Pad1.08x0.95mm_HandSolder, F.Cu at (93.3, 89.5)
- added C18: 0.1uf, Capacitor_SMD:C_0603_1608Metric_Pad1.08x0.95mm_HandSolder, F.Cu at (93.3, 92.0)
- added C19: 10uf_50V, Capacitor_SMD:C_0603_1608Metric_Pad1.08x0.95mm_HandSolder, F.Cu at (97.6, 74.5)
- added C2: 0.1uF, Capacitor_SMD:C_0603_1608Metric_Pad1.08x0.95mm_HandSolder, F.Cu at (131.6, 128.8)
- added C20: 0.1uf, Capacitor_SMD:C_0603_1608Metric_Pad1.08x0.95mm_HandSolder, F.Cu at (97.6, 77.0)
- added C21: 10uf_50V, Capacitor_SMD:C_0603_1608Metric_Pad1.08x0.95mm_HandSolder, F.Cu at (97.6, 79.5)
- added C22: 10uf, Capacitor_SMD:C_0603_1608Metric_Pad1.08x0.95mm_HandSolder, F.Cu at (97.6, 82.0)
- added C23: 0.1uf, Capacitor_SMD:C_0603_1608Metric_Pad1.08x0.95mm_HandSolder, F.Cu at (97.6, 84.5)
- added C24: 10uf, Capacitor_SMD:C_0603_1608Metric_Pad1.08x0.95mm_HandSolder, F.Cu at (97.6, 87.0)
- added C25: 0.1uf, Capacitor_SMD:C_0603_1608Metric_Pad1.08x0.95mm_HandSolder, F.Cu at (97.6, 89.5)
- added C26: 10uf_50V, Capacitor_SMD:C_0603_1608Metric_Pad1.08x0.95mm_HandSolder, F.Cu at (97.6, 92.0)
- added C27: 22uF, Capacitor_SMD:C_0603_1608Metric_Pad1.08x0.95mm_HandSolder, F.Cu at (102.0, 74.5)
- added C28: 0.1uf, Capacitor_SMD:C_0603_1608Metric_Pad1.08x0.95mm_HandSolder, F.Cu at (102.0, 77.0)
- added C29: 0.1uf, Capacitor_SMD:C_0603_1608Metric_Pad1.08x0.95mm_HandSolder, F.Cu at (102.0, 79.5)
- added C3: 0.1uF, Capacitor_SMD:C_0603_1608Metric_Pad1.08x0.95mm_HandSolder, F.Cu at (131.6, 131.3)
- added C30: 0.1uf, Capacitor_SMD:C_0603_1608Metric_Pad1.08x0.95mm_HandSolder, F.Cu at (102.0, 82.0)
- added C31: 0.1uf, Capacitor_SMD:C_0603_1608Metric_Pad1.08x0.95mm_HandSolder, F.Cu at (102.0, 84.5)
- added C32: 0.1u, Capacitor_SMD:C_0603_1608Metric_Pad1.08x0.95mm_HandSolder, F.Cu at (153.1, 74.5)
- added C33: 0.1u, Capacitor_SMD:C_0603_1608Metric_Pad1.08x0.95mm_HandSolder, F.Cu at (153.1, 77.0)
- added C34: 0.1u, Capacitor_SMD:C_0603_1608Metric_Pad1.08x0.95mm_HandSolder, F.Cu at (153.1, 79.5)
- added C35: 0.1u, Capacitor_SMD:C_0603_1608Metric_Pad1.08x0.95mm_HandSolder, F.Cu at (153.1, 82.0)
- added C36: 0.1u, Capacitor_SMD:C_0603_1608Metric_Pad1.08x0.95mm_HandSolder, F.Cu at (153.1, 84.5)
- added C37: 0.1uF, Capacitor_SMD:C_0603_1608Metric_Pad1.08x0.95mm_HandSolder, F.Cu at (140.3, 126.3)
- added C38: 0.1uF, Capacitor_SMD:C_0603_1608Metric_Pad1.08x0.95mm_HandSolder, F.Cu at (140.3, 128.8)
- added C39: 0.1uF, Capacitor_SMD:C_0603_1608Metric_Pad1.08x0.95mm_HandSolder, F.Cu at (140.3, 131.3)
- added C4: 0.1uF, Capacitor_SMD:C_0603_1608Metric_Pad1.08x0.95mm_HandSolder, F.Cu at (131.6, 133.8)
- added C40: 0.1uF, Capacitor_SMD:C_0603_1608Metric_Pad1.08x0.95mm_HandSolder, F.Cu at (140.3, 133.8)
- added C41: 0.1uF, Capacitor_SMD:C_0603_1608Metric_Pad1.08x0.95mm_HandSolder, F.Cu at (140.3, 136.3)
- added C5: 0.1uF, Capacitor_SMD:C_0603_1608Metric_Pad1.08x0.95mm_HandSolder, F.Cu at (131.6, 136.3)
- added C6: 0.1uF, Capacitor_SMD:C_0603_1608Metric_Pad1.08x0.95mm_HandSolder, F.Cu at (135.9, 126.3)
- added C7: 0.1uF, Capacitor_SMD:C_0603_1608Metric_Pad1.08x0.95mm_HandSolder, F.Cu at (135.9, 128.8)
- added C8: 0.1uF, Capacitor_SMD:C_0603_1608Metric_Pad1.08x0.95mm_HandSolder, F.Cu at (135.9, 131.3)
- added C9: 0.1uF, Capacitor_SMD:C_0603_1608Metric_Pad1.08x0.95mm_HandSolder, F.Cu at (135.9, 133.8)
- added D1: LED 0805, LED_SMD:LED_0805_2012Metric_Pad1.15x1.40mm_HandSolder, F.Cu at (124.1, 110.0)
- added D2: LED 0805, LED_SMD:LED_0805_2012Metric_Pad1.15x1.40mm_HandSolder, F.Cu at (124.1, 113.0)
- added D3: LED, LED_SMD:LED_0805_2012Metric, F.Cu at (162.4, 96.8)
- added D5: PMEG4010ET, Package_TO_SOT_SMD:SOT-23, F.Cu at (157.7, 90.1)
- added D6: PMEG4010ET, Package_TO_SOT_SMD:SOT-23, F.Cu at (124.2, 116.9)
- added FB1: FerriteBead, Ferrite_THT:LairdTech_28C0236-0JW-10, F.Cu at (114.7, 97.8)
- added FB2: FerriteBead, Ferrite_THT:LairdTech_28C0236-0JW-10, F.Cu at (114.7, 106.7)
- added FB3: FerriteBead, Ferrite_THT:LairdTech_28C0236-0JW-10, F.Cu at (114.7, 115.6)
- added FID1: Fiducial, Fiducial:Fiducial_1mm_Mask2mm, F.Cu at (171.5, 75.0)
- added FID2: Fiducial, Fiducial:Fiducial_1mm_Mask2mm, F.Cu at (171.5, 78.5)
- added FID3: Fiducial, Fiducial:Fiducial_1mm_Mask2mm, F.Cu at (171.5, 82.1)
- added FID4: Fiducial, Fiducial:Fiducial_1mm_Mask2mm, F.Cu at (171.5, 85.7)
- added J1: USB_B, Connector_USB:USB_B_OST_USB-B1HSxx_Horizontal, F.Cu at (111.4, 80.8)
- added J2: Conn_01x06_MountingPin, MountingHole:MountingHole_2.1mm, F.Cu at (171.7, 90.5)
- added J6: DC37_Receptacle_MountingHoles, Connector_Dsub:DSUB-37_Female_Horizontal_P2.77x2.84mm_EdgePinOffset7.70mm_Housed_MountingHolesOffset9.12mm, F.Cu at (151.8, 53.1)
- added Q1: BSS138, Package_TO_SOT_SMD:SOT-23_Handsoldering, F.Cu at (132.6, 75.7)
- added Q10: BSS138, Package_TO_SOT_SMD:SOT-23_Handsoldering, F.Cu at (132.6, 104.4)
- added Q11: Q_PMOS_GSD, Package_TO_SOT_SMD:SOT-23_Handsoldering, F.Cu at (132.6, 109.2)
- added Q12: BSS138, Package_TO_SOT_SMD:SOT-23_Handsoldering, F.Cu at (118.0, 138.9)
- added Q13: BSS138, Package_TO_SOT_SMD:SOT-23_Handsoldering, F.Cu at (118.0, 143.7)
- added Q14: BSS138, Package_TO_SOT_SMD:SOT-23_Handsoldering, F.Cu at (118.0, 148.5)
- added Q2: Q_PMOS_GSD, Package_TO_SOT_SMD:SOT-23_Handsoldering, F.Cu at (132.6, 80.5)
- added Q3: BSS138, Package_TO_SOT_SMD:SOT-23_Handsoldering, F.Cu at (132.6, 85.3)
- added Q4: Q_PMOS_GSD, Package_TO_SOT_SMD:SOT-23_Handsoldering, F.Cu at (132.6, 90.0)
- added Q5: BSS138, Package_TO_SOT_SMD:SOT-23_Handsoldering, F.Cu at (132.6, 94.8)
- added Q6: Q_PMOS_GSD, Package_TO_SOT_SMD:SOT-23_Handsoldering, F.Cu at (132.6, 99.6)
- added Q7: BSS138, Package_TO_SOT_SMD:SOT-23_Handsoldering, F.Cu at (118.0, 124.6)
- added Q8: BSS138, Package_TO_SOT_SMD:SOT-23_Handsoldering, F.Cu at (118.0, 129.4)
- added Q9: BSS138, Package_TO_SOT_SMD:SOT-23_Handsoldering, F.Cu at (118.0, 134.1)
- added R1: 10k, Resistor_SMD:R_0603_1608Metric_Pad0.98x0.95mm_HandSolder, F.Cu at (138.0, 74.5)
- added R10: 100, Resistor_SMD:R_0603_1608Metric_Pad0.98x0.95mm_HandSolder, F.Cu at (158.9, 114.7)
- added R11: 1.5k, Resistor_SMD:R_0603_1608Metric_Pad0.98x0.95mm_HandSolder, F.Cu at (123.4, 123.3)
- added R12: 1.5k, Resistor_SMD:R_0603_1608Metric_Pad0.98x0.95mm_HandSolder, F.Cu at (123.4, 125.9)
- added R13: 1.5k, Resistor_SMD:R_0603_1608Metric_Pad0.98x0.95mm_HandSolder, F.Cu at (123.4, 128.4)
- added R14: 180, Resistor_SMD:R_0603_1608Metric_Pad0.98x0.95mm_HandSolder, F.Cu at (102.0, 87.0)
- added R15: 180, Resistor_SMD:R_0603_1608Metric_Pad0.98x0.95mm_HandSolder, F.Cu at (102.0, 89.5)
- added R16: 180, Resistor_SMD:R_0603_1608Metric_Pad0.98x0.95mm_HandSolder, F.Cu at (102.0, 92.0)
- added R17: 1.5k, Resistor_SMD:R_0603_1608Metric_Pad0.98x0.95mm_HandSolder, F.Cu at (123.4, 130.9)
- added R18: 180, Resistor_SMD:R_0603_1608Metric_Pad0.98x0.95mm_HandSolder, F.Cu at (106.3, 74.5)
- added R19: 10k, Resistor_SMD:R_0603_1608Metric_Pad0.98x0.95mm_HandSolder, F.Cu at (158.9, 117.2)
- added R2: 10k, Resistor_SMD:R_0603_1608Metric_Pad0.98x0.95mm_HandSolder, F.Cu at (138.0, 77.0)
- added R20: 1500, Resistor_SMD:R_0603_1608Metric_Pad0.98x0.95mm_HandSolder, F.Cu at (106.3, 77.0)
- added R21: 1500, Resistor_SMD:R_0603_1608Metric_Pad0.98x0.95mm_HandSolder, F.Cu at (106.3, 79.5)
- added R22: 1.7k, Resistor_SMD:R_0603_1608Metric_Pad0.98x0.95mm_HandSolder, F.Cu at (106.3, 82.0)
- added R23: 27, Resistor_SMD:R_0603_1608Metric_Pad0.98x0.95mm_HandSolder, F.Cu at (106.3, 84.5)
- added R24: 27, Resistor_SMD:R_0603_1608Metric_Pad0.98x0.95mm_HandSolder, F.Cu at (106.3, 87.0)
- added R25: R, Resistor_SMD:R_0603_1608Metric_Pad0.98x0.95mm_HandSolder, F.Cu at (153.1, 87.0)
- added R26: 10k, Resistor_SMD:R_0603_1608Metric_Pad0.98x0.95mm_HandSolder, F.Cu at (153.1, 89.5)
- added R27: 1.5k, Resistor_SMD:R_0603_1608Metric_Pad0.98x0.95mm_HandSolder, F.Cu at (123.4, 133.4)
- added R28: 1.5k, Resistor_SMD:R_0603_1608Metric_Pad0.98x0.95mm_HandSolder, F.Cu at (123.4, 135.9)
- added R29: 1500, Resistor_SMD:R_0603_1608Metric_Pad0.98x0.95mm_HandSolder, F.Cu at (106.3, 89.5)
- added R3: 1.5k, Resistor_SMD:R_0603_1608Metric_Pad0.98x0.95mm_HandSolder, F.Cu at (138.0, 79.5)
- added R30: 10k, Resistor_SMD:R_0603_1608Metric_Pad0.98x0.95mm_HandSolder, F.Cu at (153.1, 92.0)
- added R31: 10k, Resistor_SMD:R_0603_1608Metric_Pad0.98x0.95mm_HandSolder, F.Cu at (158.9, 119.7)
- added R32: 100, Resistor_SMD:R_0603_1608Metric_Pad0.98x0.95mm_HandSolder, F.Cu at (158.9, 122.2)
- added R33: 1.5k, Resistor_SMD:R_0805_2012Metric_Pad1.20x1.40mm_HandSolder, F.Cu at (92.5, 133.0)
- added R34: 100, Resistor_SMD:R_0603_1608Metric_Pad0.98x0.95mm_HandSolder, F.Cu at (158.9, 124.7)
- added R35: 10k, Resistor_SMD:R_0603_1608Metric_Pad0.98x0.95mm_HandSolder, F.Cu at (158.9, 127.2)
- added R36: 100, Resistor_SMD:R_0603_1608Metric_Pad0.98x0.95mm_HandSolder, F.Cu at (158.9, 129.7)
- added R37: 1.5k, Resistor_SMD:R_0805_2012Metric_Pad1.20x1.40mm_HandSolder, F.Cu at (108.0, 139.5)
- added R38: 10k, Resistor_SMD:R_0603_1608Metric_Pad0.98x0.95mm_HandSolder, F.Cu at (98.9, 136.0)
- added R39: 10k, Resistor_SMD:R_0603_1608Metric_Pad0.98x0.95mm_HandSolder, F.Cu at (146.7, 77.0)
- added R4: 1.5k, Resistor_SMD:R_0603_1608Metric_Pad0.98x0.95mm_HandSolder, F.Cu at (138.0, 82.0)
- added R40: 10k, Resistor_SMD:R_0603_1608Metric_Pad0.98x0.95mm_HandSolder, F.Cu at (146.7, 79.5)
- added R41: 1.5k, Resistor_SMD:R_0603_1608Metric_Pad0.98x0.95mm_HandSolder, F.Cu at (146.7, 82.0)
- added R42: 10k, Resistor_SMD:R_0603_1608Metric_Pad0.98x0.95mm_HandSolder, F.Cu at (103.1, 144.0)
- added R43: 1.5k, Resistor_SMD:R_0805_2012Metric_Pad1.20x1.40mm_HandSolder, F.Cu at (90.0, 138.5)
- added R44: 1.5k, Resistor_SMD:R_0805_2012Metric_Pad1.20x1.40mm_HandSolder, F.Cu at (90.0, 144.0)
- added R45: 10k, Resistor_SMD:R_0603_1608Metric_Pad0.98x0.95mm_HandSolder, F.Cu at (98.9, 141.0)
- added R46: 10k, Resistor_SMD:R_0603_1608Metric_Pad0.98x0.95mm_HandSolder, F.Cu at (98.9, 143.5)
- added R47: 100, Resistor_SMD:R_0603_1608Metric_Pad0.98x0.95mm_HandSolder, F.Cu at (163.3, 114.7)
- added R48: 100, Resistor_SMD:R_0603_1608Metric_Pad0.98x0.95mm_HandSolder, F.Cu at (163.3, 117.2)
- added R49: 10k, Resistor_SMD:R_0603_1608Metric_Pad0.98x0.95mm_HandSolder, F.Cu at (163.3, 119.7)
- added R5: 10k, Resistor_SMD:R_0603_1608Metric_Pad0.98x0.95mm_HandSolder, F.Cu at (142.4, 74.5)
- added R50: 100, Resistor_SMD:R_0603_1608Metric_Pad0.98x0.95mm_HandSolder, F.Cu at (163.3, 122.2)
- added R51: 10k, Resistor_SMD:R_0603_1608Metric_Pad0.98x0.95mm_HandSolder, F.Cu at (163.3, 124.7)
- added R52: 100, Resistor_SMD:R_0603_1608Metric_Pad0.98x0.95mm_HandSolder, F.Cu at (163.3, 127.2)
- added R53: 10k, Resistor_SMD:R_0603_1608Metric_Pad0.98x0.95mm_HandSolder, F.Cu at (163.3, 129.7)
- added R54: 100, Resistor_SMD:R_0603_1608Metric_Pad0.98x0.95mm_HandSolder, F.Cu at (167.6, 114.7)
- added R55: 100, Resistor_SMD:R_0603_1608Metric_Pad0.98x0.95mm_HandSolder, F.Cu at (167.6, 117.2)
- added R56: 100, Resistor_SMD:R_0603_1608Metric_Pad0.98x0.95mm_HandSolder, F.Cu at (167.6, 119.7)
- added R57: 100, Resistor_SMD:R_0603_1608Metric_Pad0.98x0.95mm_HandSolder, F.Cu at (167.6, 122.2)
- added R6: 10k, Resistor_SMD:R_0603_1608Metric_Pad0.98x0.95mm_HandSolder, F.Cu at (142.4, 77.0)
- added R7: 1.5k, Resistor_SMD:R_0603_1608Metric_Pad0.98x0.95mm_HandSolder, F.Cu at (142.4, 79.5)
- added R8: 10k, Resistor_SMD:R_0603_1608Metric_Pad0.98x0.95mm_HandSolder, F.Cu at (142.4, 82.0)
- added R9: 10k, Resistor_SMD:R_0603_1608Metric_Pad0.98x0.95mm_HandSolder, F.Cu at (146.7, 74.5)
- added TP1: TestPoint, TestPoint:TestPoint_THTPad_D3.0mm_Drill1.5mm, F.Cu at (124.2, 95.8)
- added TP13: TestPoint, TestPoint:TestPoint_THTPad_D3.0mm_Drill1.5mm, F.Cu at (124.2, 100.9)
- added TP14: TestPoint, TestPoint:TestPoint_THTPad_D3.0mm_Drill1.5mm, F.Cu at (124.2, 105.9)
- added TP30: TestPoint, TestPoint:TestPoint_THTPad_D3.0mm_Drill1.5mm, F.Cu at (171.3, 96.0)
- added U1: ICL3232, Package_SO:SOIC-16_3.9x9.9mm_P1.27mm, F.Cu at (133.6, 119.3)
- added U10: LM7805_TO220, Package_TO_SOT_THT:TO-220-3_Vertical, F.Cu at (71.4, 100.5)
- added U11: LD39150DT33, Package_TO_SOT_SMD:TO-252-3_TabPin2, F.Cu at (98.0, 109.1)
- added U12: HCPL-2630, Package_DIP:DIP-8_W7.62mm, F.Cu at (103.6, 95.4)
- added U13: MCP111T, Package_TO_SOT_SMD:TSOT-23, F.Cu at (157.7, 94.7)
- added U14: 74AHCT1G126, Package_TO_SOT_SMD:SOT-23-5_HandSoldering, F.Cu at (172.7, 125.4)
- added U15: 74AHCT1G126, Package_TO_SOT_SMD:SOT-23-5_HandSoldering, F.Cu at (172.7, 130.2)
- added U16: 74AHCT1G126, Package_TO_SOT_SMD:SOT-23-5_HandSoldering, F.Cu at (172.7, 135.0)
- added U17: 74AHCT1G126, Package_TO_SOT_SMD:SOT-23-5_HandSoldering, F.Cu at (172.7, 139.8)
- added U19: 74LCX244, Package_SO:SOIC-16_3.9x9.9mm_P1.27mm, F.Cu at (161.0, 136.9)
- added U2: ICL3232, Package_SO:SOIC-16_3.9x9.9mm_P1.27mm, F.Cu at (142.1, 119.3)
- added U3: 74AHCT1G126, Package_TO_SOT_SMD:SOT-23-5_HandSoldering, F.Cu at (172.7, 115.9)
- added U30: PIC18F45K50_QFP, Package_QFP:TQFP-44_10x10mm_P0.8mm, F.Cu at (162.5, 80.5)
- added U4: HCPL-2630, Package_DIP:DIP-8_W7.62mm, F.Cu at (71.7, 115.0)
- added U5: HCPL-2630, Package_DIP:DIP-8_W7.62mm, F.Cu at (95.2, 126.3)
- added U6: ICL3232, Package_SO:SOIC-16_3.9x9.9mm_P1.27mm, F.Cu at (150.5, 119.3)
- added U7: 74AHCT1G126, Package_TO_SOT_SMD:SOT-23-5_HandSoldering, F.Cu at (172.7, 120.7)
- added U8: FT231XS, Package_SO:SSOP-20_3.9x8.7mm_P0.635mm, F.Cu at (107.2, 110.2)
- added U9: HCPL-2630, Package_DIP:DIP-8_W7.62mm, F.Cu at (92.7, 95.4)
- added Y1: ASV-xxxMHz, Oscillator:Oscillator_SMD_Abracon_ASV-4Pin_7.0x5.1mm, F.Cu at (164.5, 91.5)
